File: hardware/FM-1.2.1.brd (EAGLE design)
At the start: 181 x 106 mm, 120 parts, among them IC1 7805TV, IC2 MCP6004, IC3 TL072D, IC4 MCP6004, IC9 LM4040, T1 BC547, T4.1 TEENSY4.1

Commit message: Update to v1.2.1
Parts:
- added PAD1, PAD2, PAD3, PAD4: (no value), wirepad:1,6/0,9
- T1: value BC547 -> BC550
Connections:
- net D+: now also PAD3.1
- net D-: now also PAD2.1
- net GND: now also FC1.P$3, FC2.P$1, FC3.P$1, FC4.P$1, LEVEL1.P$1, LEVEL2.P$1, LEVEL3.P$1, LEVEL4.P$1, PAD4.1; no longer FC1.P$1, FC2.P$3, FC3.P$3, FC4.P$3, LEVEL1.P$3, LEVEL2.P$3, LEVEL3.P$3, LEVEL4.P$3
- net VCC: now also FC1.P$1, FC2.P$3, FC3.P$3, FC4.P$3, LEVEL1.P$3, LEVEL2.P$3, LEVEL3.P$3, LEVEL4.P$3; no longer FC1.P$3, FC2.P$1, FC3.P$1, FC4.P$1, LEVEL1.P$1, LEVEL2.P$1, LEVEL3.P$1, LEVEL4.P$1
Routing:
- net GND: track 0.00 -> 994.0 mm, vias 0 -> 2
- net N$49: track 178.4 -> 129.6 mm, vias 1 -> 2
- net VCC: track 497.8 -> 537.5 mm
- net A8: track 155.2 -> 186.2 mm, vias 5 -> 0
- net A2: track 107.8 -> 79.4 mm, vias 1 -> 2
- net -10V: track 167.8 -> 193.4 mm, vias 4 -> 2
- net D1: track 85.9 -> 110.4 mm, vias 1 -> 0
- net N$55: track 118.6 -> 140.9 mm, vias 1 -> 0
- net N$22: track 89.4 -> 109.0 mm, vias 2 -> 0
- net A11: track 181.3 -> 162.7 mm, vias 2 -> 3
- net A9: track 151.9 -> 166.0 mm, vias 2 -> 4
- net +5V: track 156.0 -> 169.9 mm, vias 3 -> 0
- net D12: track 71.6 -> 59.9 mm, vias 1 -> 0
- net D2: track 72.3 -> 60.5 mm
- net D5: track 38.8 -> 27.8 mm
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