File: hardware/FM-1.2.1.sch (EAGLE design)
At the start: 120 parts, among them IC1 7805TV, IC2 MCP6004, IC3 TL072D, IC4 MCP6004, IC9 LM4040, T1 BC547, T4.1 TEENSY4.1

Commit message: Update to v1.2.1
Parts:
- added PAD1, PAD2, PAD3, PAD4: (no value), wirepad:1,6/0,9
- T1: value BC547 -> BC550
Connections:
- net D+: now also PAD3.P
- net D-: now also PAD2.P
- net GND: now also FC1.A, FC2.E, FC3.E, FC4.E, LEVEL1.1, LEVEL2.1, LEVEL3.1, LEVEL4.1, PAD4.P; no longer FC1.E, FC2.A, FC3.A, FC4.A, LEVEL1.3, LEVEL2.3, LEVEL3.3, LEVEL4.3
- net VCC: now also FC1.E, FC2.A, FC3.A, FC4.A, LEVEL1.3, LEVEL2.3, LEVEL3.3, LEVEL4.3; no longer FC1.A, FC2.E, FC3.E, FC4.E, LEVEL1.1, LEVEL2.1, LEVEL3.1, LEVEL4.1
Other:
- moved on the sheet: FC1, USBHOST
